File: eagle/main.sch (EAGLE design)
At the start: 34 parts, among them Q1 BSS97, Q2 BSS97, Q3 BSS97, Q4 BSS97, U1 LTC3789EGNPBF

Commit message: [ update ] sch
Parts:
- removed D1, D2: 1N4148DO35-10, diode:1N4148DO35-10
- removed R12, R2: 0.01, resistor:R-EU_R1206
- added C10, C12, C13: 0.22u, rcl:C-EUC1206K
- added C9: 2.2u, rcl:C-EUC1206K
- added D5, D6: 1N4148DO35-10, diode:1N4148DO35-10
Connections:
- removed net IOSENSE+_NC: R8.2, R9.1
- removed net N$11: D4.C, L1.1, Q1.S, Q2.D
- removed net N$6: C5.1, D1.A, D2.A, U1.INTVCC
- removed net N$8: D3.A, L1.2, Q3.D, Q4.S
- removed net SENSE+_NC: R4.1, R5.2
- new net INTVCC: C5.1, D5.A, D6.A, U1.INTVCC
- new net RUN: U1.RUN
- net BOOST1: now also C12.2, D5.C; no longer D1.C
- net BOOST2: now also C10.1, C13.2, D6.C; no longer D2.C
- net GND: now also R4.1, R5.2; no longer R12.1, R4.2, R6.2
- net IOSENSE+: now also C9.2, R7.1; no longer R8.1
- net IOSENSE-: now also C9.1, R8.1; no longer R7.1
- net N$7: now also R7.2, R9.1; no longer R2.1
- net N$9: now also R4.2, R6.2; no longer R12.2
- net SENSE+: now also R6.1; no longer R5.1
- net SENSE-: now also R5.1; no longer R6.1
- net SW1: now also C12.1, D4.C, L1.1, Q1.S, Q2.D
- net SW2: now also C10.2, C13.1, D3.A, L1.2, Q3.D, Q4.S
- net VOUT: now also R8.2; no longer R2.2, R7.2
Other:
- note added: "TODO: check R12"
- note removed: "TODO: check R4"
- note removed: "TODO: choose D1"
- note removed: "TODO: choose D2"
- note removed: "TODO: connect IOSENSE+_NC"
- note removed: "TODO: connect SENSE+_NC"
- moved on the sheet: C1, C4, C6, C7, D3, Q3, Q4, R10, R3, R4, R5, R6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

Commit message: [ update ] sch
Parts:
- removed C10: 0.22u, rcl:C-EUC1206K
- removed C9: 2.2u, rcl:C-EUC1206K
- removed R7, R8: 100, resistor:R-EU_R1206
- removed R9: 0.01, resistor:R-EU_R1206
Connections:
- removed net IOSENSE+: C9.2, R7.1, U1.IOSENSE+
- removed net IOSENSE-: C9.1, R8.1, U1.IOSENSE-
- removed net N$7: C6.1, D3.C, Q4.D, R7.2, R9.1
- net BOOST2: no longer C10.1
- net SW2: no longer C10.2
- net VOUT: now also C6.1, D3.C, Q4.D, U1.IOSENSE+, U1.IOSENSE-; no longer R8.2, R9.2
Other:
- note removed: "TODO: check R12"
- note removed: "TODO: check R9"
- moved on the sheet: C13, C6, C7

Commit message: [ update ] sch
Parts:
- L1: value (none) -> 6.8u; device rcl:L-EUL2012C -> WE-HCC:WE-HCC-7443320680_1210
Connections:
- net SW1: now also L1.2; no longer L1.1
- net SW2: now also L1.1; no longer L1.2
Changed lines of the file:
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@@
 <layer number="48" name="Document" color="7" fill="1" visible="no" active="no"/>
 <layer number="49" name="Reference" color="7" fill="1" visible="no" active="no"/>
+<layer number="50" name="dxf" color="7" fill="1" visible="no" active="no"/>
 <layer number="51" name="tDocu" color="7" fill="1" visible="no" active="no"/>
 <layer number="52" name="bDocu" color="7" fill="1" visible="no" active="no"/>
+<layer number="53" name="tPadExt" color="7" fill="1" visible="no" active="no"/>
+<layer number="54" name="bPadExt" color="1" fill="1" visible="no" active="no"/>
 <layer number="91" name="Nets" color="2" fill="1" visible="yes" active="yes"/>
 <layer number="92" name="Busses" color="1" fill="1" visible="yes" active="yes"/>
@@
 <layer number="97" name="Info" color="4" fill="1" visible="yes" active="yes"/>
 <layer number="98" name="Guide" color="6" fill="1" visible="yes" active="yes"/>
+<layer number="250" name="Descript" color="3" fill="1" visible="no" active="no"/>
+<layer number="251" name="SMDround" color="12" fill="11" visible="no" active="no"/>
 </layers>
 <schematic xreflabel="%F%N/%S.%C%R" xrefpart="/%S.%C%R">
@@
 <part name="Q3" library="transistor-fet" deviceset="BSS97" device=""/>
 <part name="Q4" library="transistor-fet" deviceset="BSS97" device=""/>
-<part name="L1" library="rcl" deviceset="L-EU" device="L2012C"/>
 <part name="C6" library="rcl" deviceset="C-EU" device="C1206K" value="2.2u"/>
 <part name="C7" library="rcl" deviceset="CPOL-EU" device="A" value="330u"/>
@@
 <part name="R5" library="resistor" deviceset="R-EU_" device="R1206" value="1K"/>
 <part name="R6" library="resistor" deviceset="R-EU_" device="R1206" value="1K"/>
+<part name="L1" library="WE-HCC" deviceset="WE-HCC" device="_1210" technology="-7443320680" value="6.8u"/>
 </parts>
 <sheets>
@@
 <instance part="Q3" gate="G$1" x="134.62" y="5.08" rot="MR180"/>
 <instance part="Q4" gate="G$1" x="134.62" y="-17.78" rot="MR180"/>
-<instance part="L1" gate="G$1" x="151.13" y="33.02"/>
 <instance part="C6" gate="G$1" x="157.48" y="-5.08" smashed="yes" rot="R180">
 <attribute name="NAME" x="155.956" y="-0.381" size="1.778" layer="95" align="top-right"/>
@@
 <instance part="R5" gate="G$1" x="115.57" y="21.59"/>
 <instance part="R6" gate="G$1" x="115.57" y="13.97"/>
+<instance part="L1" gate="G$1" x="151.13" y="33.02" rot="R90"/>
 </instances>
 <busses>
@@
 <wire x1="144.78" y1="-3.81" x2="139.7" y2="-3.81" width="0.1524" layer="91"/>
 <junction x="139.7" y="-3.81"/>
-<pinref part="L1" gate="G$1" pin="2"/>
 <wire x1="151.13" y1="27.94" x2="151.13" y2="-3.81" width="0.1524" layer="91"/>
 <wire x1="151.13" y1="-3.81" x2="144.78" y2="-3.81" width="0.1524" layer="91"/>
@@
 <junction x="144.78" y="-3.81"/>
 <junction x="139.7" y="-3.81"/>
+<pinref part="L1" gate="G$1" pin="1"/>
 </segment>
 <segment>
@@
 <wire x1="144.78" y1="40.64" x2="151.13" y2="40.64" width="0.1524" layer="91"/>
 <junction x="144.78" y="40.64"/>
-<pinref part="L1" gate="G$1" pin="1"/>
 <wire x1="151.13" y1="40.64" x2="151.13" y2="38.1" width="0.1524" layer="91"/>
 <wire x1="139.7" y1="40.64" x2="119.38" y2="40.64" width="0.1524" layer="91"/>
 <label x="119.38" y="40.64" size="1.778" layer="95"/>
-</segment>
-<segment>
+<pinref part="L1" gate="G$1" pin="2"/>
+</segment>
+<segment>

Commit message: [ update ] sch
Other:
- note added: "TODO: connect RUN to switch"
Changed lines of the file:
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@@
 <text x="45.72" y="128.27" size="1.778" layer="97">TODO: choose C4</text>
 <text x="125.73" y="116.84" size="1.778" layer="97">TODO: choose C5</text>
+<text x="16.51" y="53.34" size="1.778" layer="97">TODO: connect RUN to switch</text>
 </plain>
 <instances>

Commit message: [ update, add ] eagle/main.brd
Other:
- note added: "TODO: si4840bdy"
- note added: "TODO: sqj886ep-t1-ge3"
Changed lines of the file:
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@@
 <setting verticaltext="up"/>
 </settings>
-<grid distance="1.27" unitdist="mm" unit="mm" style="lines" multiple="1" display="yes" altdistance="0.01" altunitdist="inch" altunit="inch"/>
+<grid distance="0.05" unitdist="inch" unit="inch" style="lines" multiple="1" display="yes" altdistance="0.01" altunitdist="inch" altunit="inch"/>
 <layers>
 <layer number="1" name="Top" color="4" fill="1" visible="no" active="no"/>
@@
 <layer number="53" name="tPadExt" color="7" fill="1" visible="no" active="no"/>
 <layer number="54" name="bPadExt" color="1" fill="1" visible="no" active="no"/>
+<layer number="56" name="wert" color="7" fill="1" visible="no" active="no"/>
 <layer number="91" name="Nets" color="2" fill="1" visible="yes" active="yes"/>
 <layer number="92" name="Busses" color="1" fill="1" visible="yes" active="yes"/>
@@
 <layer number="97" name="Info" color="4" fill="1" visible="yes" active="yes"/>
 <layer number="98" name="Guide" color="6" fill="1" visible="yes" active="yes"/>
+<layer number="99" name="SpiceOrder" color="7" fill="1" visible="yes" active="yes"/>
 <layer number="250" name="Descript" color="3" fill="1" visible="no" active="no"/>
 <layer number="251" name="SMDround" color="12" fill="11" visible="no" active="no"/>
@@
 <text x="125.73" y="116.84" size="1.778" layer="97">TODO: choose C5</text>
 <text x="16.51" y="53.34" size="1.778" layer="97">TODO: connect RUN to switch</text>
+<text x="173.99" y="46.99" size="1.778" layer="97">TODO: sqj886ep-t1-ge3</text>
+<text x="173.99" y="33.02" size="1.778" layer="97">TODO: si4840bdy</text>
+<text x="172.72" y="5.08" size="1.778" layer="97">TODO: si4840bdy</text>
+<text x="172.72" y="-16.51" size="1.778" layer="97">TODO: si4840bdy</text>
 </plain>
 <instances>

Commit message: [ update ] sch
Parts:
- removed D5, D6: 1N4148DO35-10, diode:1N4148DO35-10
- added D1, D2: (no value), diode:DIODE-SCHOTTKY-POWER-DI-123
Connections:
- net BOOST1: now also D1.C; no longer D5.C
- net BOOST2: now also D2.C; no longer D6.C
- net INTVCC: now also D1.A, D2.A; no longer D5.A, D6.A
- net N$9: now also D3.A; no longer D4.A
- net SW1: now also D3.C; no longer D4.C
- net SW2: now also D4.A; no longer D3.A
- net VOUT: now also D4.C; no longer D3.C
Other:
- note added: "TODO: B240A"
- note added: "TODO: check package"
- moved on the sheet: D3, D4

Commit message: [ update ] sch
Parts:
- added R12: 121K, resistor:R-EU_R1206
- D3, D4: value 1N4148DO35-10 -> (none); device diode:1N4148DO35-10 -> diode:DIODE-DO214AC
- Q2, Q3, Q4: value BSS97 -> (none); device transistor-fet:BSS97 -> transistor-power:N-MOSFET-SO8S
Connections:
- new net N$6: R12.1, U1.PGOOD
- net INTVCC: now also R12.2
Other:
- note added: "NOTE: D1, D2 are DFLS160"
- note added: "NOTE: D3, D4 are B240A"
- note added: "NOTE: Q1 is SQJ886EP-T1-GE3"
- note added: "NOTE: Q2, Q3, Q4 are SI4840BDY"
- note removed: "TODO: B240A"
- note removed: "TODO: check package"
- note removed: "TODO: si4840bdy"
- moved on the sheet: D4, L1

Commit message: [ update ] sch
Parts:
- Q1: value BSS97 -> SQJ886EP; device transistor-fet:BSS97 -> transistor-fet:SQJ886EP
Other:
- note added: "TODO: q1 sqj886ep-t1-ge3 package is powerpak-so8, not powerpak-so8-l"
- note removed: "TODO: sqj886ep-t1-ge3"
Changed lines of the file:
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@@
 <part name="C4" library="rcl" deviceset="C-EU" device="C1206K" value="1u"/>
 <part name="C5" library="rcl" deviceset="C-EU" device="C1206K" value="4.7u"/>
-<part name="Q1" library="transistor-fet" deviceset="BSS97" device=""/>
 <part name="C6" library="rcl" deviceset="C-EU" device="C1206K" value="2.2u"/>
 <part name="C7" library="rcl" deviceset="CPOL-EU" device="A" value="330u"/>
@@
 <part name="Q3" library="transistor-power" deviceset="N-MOSFET-SO8" device="S"/>
 <part name="Q4" library="transistor-power" deviceset="N-MOSFET-SO8" device="S"/>
+<part name="Q1" library="transistor-fet" deviceset="SQJ886EP" device=""/>
 </parts>
 <sheets>
@@
 <text x="125.73" y="116.84" size="1.778" layer="97">TODO: choose C5</text>
 <text x="16.51" y="53.34" size="1.778" layer="97">TODO: connect RUN to switch</text>
-<text x="173.99" y="46.99" size="1.778" layer="97">TODO: sqj886ep-t1-ge3</text>
+<text x="173.99" y="46.99" size="1.778" layer="97">TODO: q1 sqj886ep-t1-ge3 package is powerpak-so8, not powerpak-so8-l</text>
 <text x="119.38" y="60.96" size="1.778" layer="97">NOTE: D3, D4 are B240A</text>
 <text x="163.83" y="121.92" size="1.778" layer="97">NOTE: D1, D2 are DFLS160</text>
@@
 <attribute name="VALUE" x="126.619" y="114.554" size="1.778" layer="96" rot="R180" align="top-right"/>
 </instance>
-<instance part="Q1" gate="G$1" x="134.62" y="48.26"/>
 <instance part="C6" gate="G$1" x="157.48" y="-5.08" smashed="yes" rot="R180">
 <attribute name="NAME" x="155.956" y="-0.381" size="1.778" layer="95" align="top-right"/>
@@
 <attribute name="NAME" x="132.08" y="-7.62" size="1.778" layer="95" rot="MR180"/>
 <attribute name="VALUE" x="142.24" y="-12.7" size="1.778" layer="96" rot="MR180"/>
+</instance>
+<instance part="Q1" gate="G$1" x="137.16" y="48.26" smashed="yes">
+<attribute name="NAME" x="134.62" y="52.07" size="1.778" layer="95"/>
 </instance>
 </instances>
@@
 <segment>
 <pinref part="C8" gate="G$1" pin="1"/>
-<pinref part="Q1" gate="G$1" pin="D"/>
-<wire x1="139.7" y1="50.8" x2="139.7" y2="55.88" width="0.1524" layer="91"/>
+<wire x1="119.38" y1="55.88" x2="139.7" y2="55.88" width="0.1524" layer="91"/>
 <wire x1="139.7" y1="55.88" x2="157.48" y2="55.88" width="0.1524" layer="91"/>
 <wire x1="157.48" y1="55.88" x2="157.48" y2="48.26" width="0.1524" layer="91"/>
-<wire x1="139.7" y1="55.88" x2="119.38" y2="55.88" width="0.1524" layer="91"/>
-<junction x="139.7" y="55.88"/>
 <wire x1="157.48" y1="55.88" x2="172.72" y2="55.88" width="0.1524" layer="91"/>
 <junction x="157.48" y="55.88"/>
 <label x="167.64" y="55.88" size="1.778" layer="95"/>
+<wire x1="139.7" y1="53.34" x2="139.7" y2="55.88" width="0.1524" layer="91"/>
+<junction x="139.7" y="55.88"/>
+<pinref part="Q1" gate="G$1" pin="D"/>
 </segment>
 </net>
@@
 </segment>
 <segment>
+<label x="119.38" y="45.72" size="1.778" layer="95"/>
 <pinref part="Q1" gate="G$1" pin="G"/>
-<wire x1="129.54" y1="45.72" x2="119.38" y2="45.72" width="0.1524" layer="91"/>
-<label x="119.38" y="45.72" size="1.778" layer="95"/>
+<wire x1="119.38" y1="45.72" x2="134.62" y2="45.72" width="0.1524" layer="91"/>
 </segment>
 </net>
@@
 </segment>
 <segment>
-<pinref part="Q1" gate="G$1" pin="S"/>
-<wire x1="139.7" y1="45.72" x2="139.7" y2="40.64" width="0.1524" layer="91"/>
 <wire x1="139.7" y1="40.64" x2="139.7" y2="38.1" width="0.1524" layer="91"/>
 <wire x1="139.7" y1="40.64" x2="144.78" y2="40.64" width="0.1524" layer="91"/>
@@
 <pinref part="D3" gate="G$1" pin="C"/>
 <pinref part="Q2" gate="G$1" pin="D"/>
-</segment>
-<segment>
+<wire x1="139.7" y1="43.18" x2="139.7" y2="40.64" width="0.1524" layer="91"/>
+<pinref part="Q1" gate="G$1" pin="S"/>
+</segment>
+<segment>
