File: eagle/main.sch (EAGLE design)
At the start: 32 parts, among them Q1 SQJ886EP, U1 LTC3789EGNPBF

Commit message: [ update ] sch
Parts:
- C7: value 330u -> 330UF; device rcl:CPOL-EUA -> Panasonic-EEEFT_EEEH:EEE-FT1H331AP-CASE-G
Connections:
- net GND: now also C7.2; no longer C7.-
- net VOUT: now also C7.1; no longer C7.+
Other:
- note removed: "TODO: choose C4"
- note removed: "TODO: choose C5"
- note removed: "TODO: choose R11"
- note removed: "TODO: select C2"
- note removed: "TODO: select C3"
Changed lines of the file:
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@@
 <part name="C5" library="rcl" deviceset="C-EU" device="C1206K" value="4.7u"/>
 <part name="C6" library="rcl" deviceset="C-EU" device="C1206K" value="2.2u"/>
-<part name="C7" library="rcl" deviceset="CPOL-EU" device="A" value="330u"/>
 <part name="C8" library="rcl" deviceset="C-EU" device="C1206K" value="47u"/>
 <part name="R4" library="resistor" deviceset="R-EU_" device="R1206" value="0.01"/>
@@
 <part name="Q4" library="transistor-power" deviceset="N-MOSFET-SO8" device="S"/>
 <part name="Q1" library="transistor-fet" deviceset="SQJ886EP" device=""/>
+<part name="C7" library="Panasonic-EEEFT_EEEH" deviceset="EEE-" device="-CASE-G" technology="FT1H331AP" value="330UF"/>
 </parts>
 <sheets>
@@
 <text x="0" y="97.79" size="1.778" layer="97">3.4V, 5.2V, 12V, 19.6V</text>
 <text x="0" y="102.87" size="1.778" layer="97">TODO: choose a switch</text>
-<text x="125.73" y="119.38" size="1.778" layer="97">TODO: choose R11</text>
-<text x="125.73" y="121.92" size="1.778" layer="97">TODO: select C2</text>
-<text x="125.73" y="124.46" size="1.778" layer="97">TODO: select C3</text>
-<text x="45.72" y="128.27" size="1.778" layer="97">TODO: choose C4</text>
-<text x="125.73" y="116.84" size="1.778" layer="97">TODO: choose C5</text>
 <text x="16.51" y="53.34" size="1.778" layer="97">TODO: connect RUN to switch</text>
-<text x="173.99" y="46.99" size="1.778" layer="97">TODO: q1 sqj886ep-t1-ge3 package is powerpak-so8, not powerpak-so8-l</text>
-<text x="119.38" y="60.96" size="1.778" layer="97">NOTE: D3, D4 are B240A</text>
-<text x="163.83" y="121.92" size="1.778" layer="97">NOTE: D1, D2 are DFLS160</text>
-<text x="119.38" y="63.5" size="1.778" layer="97">NOTE: Q2, Q3, Q4 are SI4840BDY</text>
-<text x="119.38" y="66.04" size="1.778" layer="97">NOTE: Q1 is SQJ886EP-T1-GE3</text>
+<text x="119.38" y="66.04" size="1.778" layer="97">TODO: q1 sqj886ep-t1-ge3 package is powerpak-so8, not powerpak-so8-l</text>
+<text x="119.38" y="58.42" size="1.778" layer="97">NOTE: D3, D4 are B240A</text>
+<text x="163.83" y="119.38" size="1.778" layer="97">NOTE: D1, D2 are DFLS160</text>
+<text x="119.38" y="60.96" size="1.778" layer="97">NOTE: Q2, Q3, Q4 are SI4840BDY</text>
+<text x="119.38" y="63.5" size="1.778" layer="97">NOTE: Q1 is SQJ886EP-T1-GE3</text>
 </plain>
 <instances>
@@
 <attribute name="VALUE" x="155.956" y="-5.461" size="1.778" layer="96" align="top-right"/>
 </instance>
-<instance part="C7" gate="G$1" x="165.1" y="-25.4"/>
 <instance part="C8" gate="G$1" x="157.48" y="45.72" smashed="yes">
 <attribute name="NAME" x="156.464" y="48.641" size="1.778" layer="95" align="top-right"/>
@@
 <attribute name="NAME" x="134.62" y="52.07" size="1.778" layer="95"/>
 </instance>
+<instance part="C7" gate="A" x="165.1" y="-22.86" smashed="yes" rot="R270">
+<attribute name="NAME" x="167.8686" y="-29.5656" size="2.0828" layer="95" ratio="10" rot="SR0"/>
+<attribute name="VALUE" x="168.275" y="-26.0096" size="2.0828" layer="96" ratio="10" rot="SR0"/>
+</instance>
 </instances>
 <busses>
@@
 </segment>
 <segment>
-<pinref part="C7" gate="G$1" pin="-"/>
-<wire x1="165.1" y1="-30.48" x2="165.1" y2="-33.02" width="0.1524" layer="91"/>
 <wire x1="165.1" y1="-33.02" x2="172.72" y2="-33.02" width="0.1524" layer="91"/>
 <label x="167.64" y="-33.02" size="1.778" layer="95"/>
+<pinref part="C7" gate="A" pin="2"/>
+<wire x1="165.1" y1="-33.02" x2="165.1" y2="-30.48" width="0.1524" layer="91"/>
 </segment>
 </net>
@@
 </segment>
 <segment>
-<pinref part="C7" gate="G$1" pin="+"/>
 <wire x1="165.1" y1="-20.32" x2="165.1" y2="-22.86" width="0.1524" layer="91"/>
 <wire x1="165.1" y1="-20.32" x2="172.72" y2="-20.32" width="0.1524" layer="91"/>
@@
 <pinref part="Q4" gate="G$1" pin="D"/>
 <wire x1="139.7" y1="-20.32" x2="139.7" y2="-17.78" width="0.1524" layer="91"/>
-</segment>
-<segment>
+<pinref part="C7" gate="A" pin="1"/>
+</segment>
+<segment>

Commit message: [ update ] sch
Parts:
- added C8_1, C8_2, C8_3, C8_4: 10u, rcl:C-EUC1206K
- C8_0: value 47u -> 10u
- renumbered C8 to C8_0
Connections:
- net GND: now also C8_1.2, C8_2.2, C8_3.2, C8_4.2
- net VIN: now also C8_1.1, C8_2.1, C8_3.1, C8_4.1
Changed lines of the file:
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@@
 <part name="C5" library="rcl" deviceset="C-EU" device="C1206K" value="4.7u"/>
 <part name="C6" library="rcl" deviceset="C-EU" device="C1206K" value="2.2u"/>
-<part name="C8" library="rcl" deviceset="C-EU" device="C1206K" value="47u"/>
+<part name="C8_0" library="rcl" deviceset="C-EU" device="C1206K" value="10u"/>
 <part name="R4" library="resistor" deviceset="R-EU_" device="R1206" value="0.01"/>
 <part name="C12" library="rcl" deviceset="C-EU" device="C1206K" value="0.22u"/>
@@
 <part name="Q1" library="transistor-fet" deviceset="SQJ886EP" device=""/>
 <part name="C7" library="Panasonic-EEEFT_EEEH" deviceset="EEE-" device="-CASE-G" technology="FT1H331AP" value="330UF"/>
+<part name="C8_1" library="rcl" deviceset="C-EU" device="C1206K" value="10u"/>
+<part name="C8_2" library="rcl" deviceset="C-EU" device="C1206K" value="10u"/>
+<part name="C8_3" library="rcl" deviceset="C-EU" device="C1206K" value="10u"/>
+<part name="C8_4" library="rcl" deviceset="C-EU" device="C1206K" value="10u"/>
 </parts>
 <sheets>
@@
 <attribute name="VALUE" x="155.956" y="-5.461" size="1.778" layer="96" align="top-right"/>
 </instance>
-<instance part="C8" gate="G$1" x="157.48" y="45.72" smashed="yes">
+<instance part="C8_0" gate="G$1" x="157.48" y="45.72" smashed="yes">
 <attribute name="NAME" x="156.464" y="48.641" size="1.778" layer="95" align="top-right"/>
 <attribute name="VALUE" x="156.464" y="42.291" size="1.778" layer="96" align="top-right"/>
@@
 <attribute name="VALUE" x="168.275" y="-26.0096" size="2.0828" layer="96" ratio="10" rot="SR0"/>
 </instance>
+<instance part="C8_1" gate="G$1" x="165.1" y="45.72" smashed="yes">
+<attribute name="NAME" x="164.084" y="48.641" size="1.778" layer="95" align="top-right"/>
+<attribute name="VALUE" x="164.084" y="42.291" size="1.778" layer="96" align="top-right"/>
+</instance>
+<instance part="C8_2" gate="G$1" x="172.72" y="45.72" smashed="yes">
+<attribute name="NAME" x="171.704" y="48.641" size="1.778" layer="95" align="top-right"/>
+<attribute name="VALUE" x="171.704" y="42.291" size="1.778" layer="96" align="top-right"/>
+</instance>
+<instance part="C8_3" gate="G$1" x="180.34" y="45.72" smashed="yes">
+<attribute name="NAME" x="179.324" y="48.641" size="1.778" layer="95" align="top-right"/>
+<attribute name="VALUE" x="179.324" y="42.291" size="1.778" layer="96" align="top-right"/>
+</instance>
+<instance part="C8_4" gate="G$1" x="187.96" y="45.72" smashed="yes">
+<attribute name="NAME" x="186.944" y="48.641" size="1.778" layer="95" align="top-right"/>
+<attribute name="VALUE" x="186.944" y="42.291" size="1.778" layer="96" align="top-right"/>
+</instance>
 </instances>
 <busses>
@@
 </segment>
 <segment>
-<pinref part="C8" gate="G$1" pin="2"/>
-<wire x1="157.48" y1="40.64" x2="157.48" y2="24.13" width="0.1524" layer="91"/>
+<pinref part="C8_0" gate="G$1" pin="2"/>
+<wire x1="157.48" y1="40.64" x2="157.48" y2="38.1" width="0.1524" layer="91"/>
+<wire x1="157.48" y1="38.1" x2="157.48" y2="24.13" width="0.1524" layer="91"/>
 <wire x1="157.48" y1="24.13" x2="172.72" y2="24.13" width="0.1524" layer="91"/>
 <label x="167.64" y="24.13" size="1.778" layer="95"/>
@@
 <wire x1="157.48" y1="24.13" x2="157.48" y2="0" width="0.1524" layer="91"/>
 <junction x="157.48" y="24.13"/>
+<pinref part="C8_4" gate="G$1" pin="2"/>
+<wire x1="157.48" y1="38.1" x2="165.1" y2="38.1" width="0.1524" layer="91"/>
+<wire x1="165.1" y1="38.1" x2="172.72" y2="38.1" width="0.1524" layer="91"/>
+<wire x1="172.72" y1="38.1" x2="180.34" y2="38.1" width="0.1524" layer="91"/>
+<wire x1="180.34" y1="38.1" x2="187.96" y2="38.1" width="0.1524" layer="91"/>
+<wire x1="187.96" y1="38.1" x2="187.96" y2="40.64" width="0.1524" layer="91"/>
+<junction x="157.48" y="38.1"/>
+<pinref part="C8_3" gate="G$1" pin="2"/>
+<wire x1="180.34" y1="40.64" x2="180.34" y2="38.1" width="0.1524" layer="91"/>
+<junction x="180.34" y="38.1"/>
+<pinref part="C8_2" gate="G$1" pin="2"/>
+<wire x1="172.72" y1="40.64" x2="172.72" y2="38.1" width="0.1524" layer="91"/>
+<junction x="172.72" y="38.1"/>
+<pinref part="C8_1" gate="G$1" pin="2"/>
+<wire x1="165.1" y1="40.64" x2="165.1" y2="38.1" width="0.1524" layer="91"/>
+<junction x="165.1" y="38.1"/>
 </segment>
 <segment>
@@
 </segment>
 <segment>
-<pinref part="C8" gate="G$1" pin="1"/>
+<pinref part="C8_0" gate="G$1" pin="1"/>
 <wire x1="119.38" y1="55.88" x2="139.7" y2="55.88" width="0.1524" layer="91"/>
 <wire x1="139.7" y1="55.88" x2="157.48" y2="55.88" width="0.1524" layer="91"/>
-<wire x1="157.48" y1="55.88" x2="157.48" y2="48.26" width="0.1524" layer="91"/>
+<wire x1="157.48" y1="55.88" x2="157.48" y2="50.8" width="0.1524" layer="91"/>
+<wire x1="157.48" y1="50.8" x2="157.48" y2="48.26" width="0.1524" layer="91"/>
 <wire x1="157.48" y1="55.88" x2="172.72" y2="55.88" width="0.1524" layer="91"/>
 <junction x="157.48" y="55.88"/>
@@
 <junction x="139.7" y="55.88"/>
 <pinref part="Q1" gate="G$1" pin="D"/>
+<pinref part="C8_4" gate="G$1" pin="1"/>
+<wire x1="157.48" y1="50.8" x2="165.1" y2="50.8" width="0.1524" layer="91"/>
+<wire x1="165.1" y1="50.8" x2="172.72" y2="50.8" width="0.1524" layer="91"/>
+<wire x1="172.72" y1="50.8" x2="180.34" y2="50.8" width="0.1524" layer="91"/>
+<wire x1="180.34" y1="50.8" x2="187.96" y2="50.8" width="0.1524" layer="91"/>
+<wire x1="187.96" y1="50.8" x2="187.96" y2="48.26" width="0.1524" layer="91"/>
+<junction x="157.48" y="50.8"/>
+<pinref part="C8_3" gate="G$1" pin="1"/>
+<wire x1="180.34" y1="48.26" x2="180.34" y2="50.8" width="0.1524" layer="91"/>
+<junction x="180.34" y="50.8"/>
+<pinref part="C8_2" gate="G$1" pin="1"/>
+<wire x1="172.72" y1="48.26" x2="172.72" y2="50.8" width="0.1524" layer="91"/>
+<junction x="172.72" y="50.8"/>
+<pinref part="C8_1" gate="G$1" pin="1"/>
+<wire x1="165.1" y1="48.26" x2="165.1" y2="50.8" width="0.1524" layer="91"/>
+<junction x="165.1" y="50.8"/>
 </segment>
 </net>

Commit message: [ update ] sch
Parts:
- added CON_POW_IN, CON_POW_OUT: (no value), pinhead:PINHD-1X2
- added CON_RUN: (no value), con-lstb:MA03-1
- added CON_VSEL: (no value), con-lstb:MA04-2
- added D5: BZX84, diode:BZX84
- added R13: 280K, resistor:R-EU_R1206
- added R14: 65K, resistor:R-EU_R1206
Connections:
- new net N$10: CON_VSEL.3, R2_3.1
- new net N$11: CON_RUN.2, R13.1
- new net N$7: CON_VSEL.5, R2_2.1
- new net N$8: CON_VSEL.7, R2_1.1
- net GND: now also CON_POW_IN.2, CON_POW_OUT.2, CON_RUN.1, D5.A, R14.1
- net RUN: now also D5.C, R13.2, R14.2
- net VFB: now also CON_VSEL.1, CON_VSEL.2, CON_VSEL.4, CON_VSEL.6, CON_VSEL.8; no longer R2_1.1, R2_2.1, R2_3.1
- net VIN: now also CON_POW_IN.1, CON_RUN.3
- net VOUT: now also CON_POW_OUT.1
Other:
- note removed: "TODO: choose a switch"
- note removed: "TODO: connect RUN to switch"
- moved on the sheet: R1, R2_1, R2_2, R2_3, R2_4

Commit message: [ update ] sch
Parts:
- removed CON_POW_IN, CON_POW_OUT: (no value), pinhead:PINHD-1X2
- added POW_IN, POW_OUT: (no value), con-ptr500:AK300/2
Connections:
- net GND: now also POW_IN-2.KL, POW_OUT-2.KL; no longer CON_POW_IN.2, CON_POW_OUT.2
- net VIN: now also POW_IN-1.KL; no longer CON_POW_IN.1
- net VOUT: now also POW_OUT-1.KL; no longer CON_POW_OUT.1
Changed lines of the file:
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@@
 <part name="R14" library="resistor" deviceset="R-EU_" device="R1206" value="65K"/>
 <part name="D5" library="diode" deviceset="BZX84" device=""/>
-<part name="CON_POW_IN" library="pinhead" deviceset="PINHD-1X2" device=""/>
-<part name="CON_POW_OUT" library="pinhead" deviceset="PINHD-1X2" device=""/>
+<part name="POW_IN" library="con-ptr500" deviceset="AK300/2" device=""/>
+<part name="POW_OUT" library="con-ptr500" deviceset="AK300/2" device=""/>
 </parts>
 <sheets>
@@
 <attribute name="VALUE" x="34.29" y="40.64" size="1.778" layer="96" rot="R180"/>
 </instance>
-<instance part="CON_POW_IN" gate="G$1" x="-3.81" y="19.05" smashed="yes" rot="MR0">
-<attribute name="NAME" x="11.43" y="24.765" size="1.778" layer="95" rot="MR0"/>
-<attribute name="VALUE" x="2.54" y="13.97" size="1.778" layer="96" rot="MR0"/>
-</instance>
-<instance part="CON_POW_OUT" gate="G$1" x="22.86" y="19.05" smashed="yes" rot="MR0">
-<attribute name="NAME" x="40.64" y="24.765" size="1.778" layer="95" rot="MR0"/>
-<attribute name="VALUE" x="29.21" y="13.97" size="1.778" layer="96" rot="MR0"/>
-</instance>
+<instance part="POW_IN" gate="-1" x="8.89" y="20.32"/>
+<instance part="POW_IN" gate="-2" x="8.89" y="15.24"/>
+<instance part="POW_OUT" gate="-1" x="10.16" y="5.08"/>
+<instance part="POW_OUT" gate="-2" x="10.16" y="0"/>
 </instances>
 <busses>
@@
 </segment>
 <segment>
-<pinref part="CON_POW_IN" gate="G$1" pin="2"/>
-<wire x1="-1.27" y1="19.05" x2="11.43" y2="19.05" width="0.1524" layer="91"/>
-<label x="6.35" y="19.05" size="1.778" layer="95"/>
-</segment>
-<segment>
-<pinref part="CON_POW_OUT" gate="G$1" pin="2"/>
-<wire x1="25.4" y1="19.05" x2="38.1" y2="19.05" width="0.1524" layer="91"/>
-<label x="33.02" y="19.05" size="1.778" layer="95"/>
+<pinref part="POW_IN" gate="-2" pin="KL"/>
+<wire x1="13.97" y1="15.24" x2="20.32" y2="15.24" width="0.1524" layer="91"/>
+<label x="15.24" y="15.24" size="1.778" layer="95"/>
+</segment>
+<segment>
+<pinref part="POW_OUT" gate="-2" pin="KL"/>
+<wire x1="15.24" y1="0" x2="21.59" y2="0" width="0.1524" layer="91"/>
+<label x="16.51" y="0" size="1.778" layer="95"/>
 </segment>
 </net>
@@
 </segment>
 <segment>
-<pinref part="CON_POW_OUT" gate="G$1" pin="1"/>
-<wire x1="25.4" y1="21.59" x2="38.1" y2="21.59" width="0.1524" layer="91"/>
-<label x="31.75" y="21.59" size="1.778" layer="95"/>
+<wire x1="15.24" y1="5.08" x2="21.59" y2="5.08" width="0.1524" layer="91"/>
+<label x="15.24" y="5.08" size="1.778" layer="95"/>
+<pinref part="POW_OUT" gate="-1" pin="KL"/>
 </segment>
 </net>
@@
 </segment>
 <segment>
-<pinref part="CON_POW_IN" gate="G$1" pin="1"/>
-<wire x1="-1.27" y1="21.59" x2="11.43" y2="21.59" width="0.1524" layer="91"/>
-<label x="7.62" y="21.59" size="1.778" layer="95"/>
+<pinref part="POW_IN" gate="-1" pin="KL"/>
+<wire x1="13.97" y1="20.32" x2="20.32" y2="20.32" width="0.1524" layer="91"/>
+<label x="16.51" y="20.32" size="1.778" layer="95"/>
 </segment>
 </net>

Commit message: [ update ] sch
Parts:
- renumbered POW_IN to CON_PIN, POW_OUT to CON_POUT
Changed lines of the file:
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@@
 <part name="R14" library="resistor" deviceset="R-EU_" device="R1206" value="65K"/>
 <part name="D5" library="diode" deviceset="BZX84" device=""/>
-<part name="POW_IN" library="con-ptr500" deviceset="AK300/2" device=""/>
-<part name="POW_OUT" library="con-ptr500" deviceset="AK300/2" device=""/>
+<part name="CON_PIN" library="con-ptr500" deviceset="AK300/2" device=""/>
+<part name="CON_POUT" library="con-ptr500" deviceset="AK300/2" device=""/>
 </parts>
 <sheets>
@@
 <attribute name="VALUE" x="34.29" y="40.64" size="1.778" layer="96" rot="R180"/>
 </instance>
-<instance part="POW_IN" gate="-1" x="8.89" y="20.32"/>
-<instance part="POW_IN" gate="-2" x="8.89" y="15.24"/>
-<instance part="POW_OUT" gate="-1" x="10.16" y="5.08"/>
-<instance part="POW_OUT" gate="-2" x="10.16" y="0"/>
+<instance part="CON_PIN" gate="-1" x="8.89" y="20.32"/>
+<instance part="CON_PIN" gate="-2" x="8.89" y="15.24"/>
+<instance part="CON_POUT" gate="-1" x="10.16" y="5.08"/>
+<instance part="CON_POUT" gate="-2" x="10.16" y="0"/>
 </instances>
 <busses>
@@
 </segment>
 <segment>
-<pinref part="POW_IN" gate="-2" pin="KL"/>
+<pinref part="CON_PIN" gate="-2" pin="KL"/>
 <wire x1="13.97" y1="15.24" x2="20.32" y2="15.24" width="0.1524" layer="91"/>
 <label x="15.24" y="15.24" size="1.778" layer="95"/>
 </segment>
 <segment>
-<pinref part="POW_OUT" gate="-2" pin="KL"/>
+<pinref part="CON_POUT" gate="-2" pin="KL"/>
 <wire x1="15.24" y1="0" x2="21.59" y2="0" width="0.1524" layer="91"/>
 <label x="16.51" y="0" size="1.778" layer="95"/>
@@
 <wire x1="15.24" y1="5.08" x2="21.59" y2="5.08" width="0.1524" layer="91"/>
 <label x="15.24" y="5.08" size="1.778" layer="95"/>
-<pinref part="POW_OUT" gate="-1" pin="KL"/>
+<pinref part="CON_POUT" gate="-1" pin="KL"/>
 </segment>
 </net>
@@
 </segment>
 <segment>
-<pinref part="POW_IN" gate="-1" pin="KL"/>
+<pinref part="CON_PIN" gate="-1" pin="KL"/>
 <wire x1="13.97" y1="20.32" x2="20.32" y2="20.32" width="0.1524" layer="91"/>
 <label x="16.51" y="20.32" size="1.778" layer="95"/>

Commit message: [ update ] sch
Changed lines of the file:
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@@
 <part name="C6" library="rcl" deviceset="C-EU" device="C1206K" value="2.2u"/>
 <part name="C8_0" library="rcl" deviceset="C-EU" device="C1206K" value="10u"/>
-<part name="R4" library="resistor" deviceset="R-EU_" device="R1206" value="0.01"/>
 <part name="C12" library="rcl" deviceset="C-EU" device="C1206K" value="0.22u"/>
 <part name="C13" library="rcl" deviceset="C-EU" device="C1206K" value="0.22u"/>
@@
 <part name="CON_PIN" library="con-ptr500" deviceset="AK300/2" device=""/>
 <part name="CON_POUT" library="con-ptr500" deviceset="AK300/2" device=""/>
+<part name="R4" library="resistor" deviceset="R-EU_" device="R1206" value="0.01"/>
 </parts>
 <sheets>
@@
 <attribute name="VALUE" x="156.464" y="42.291" size="1.778" layer="96" align="top-right"/>
 </instance>
-<instance part="R4" gate="G$1" x="132.08" y="24.13"/>
 <instance part="C12" gate="G$1" x="173.99" y="114.3" smashed="yes" rot="R90">
 <attribute name="NAME" x="169.799" y="115.824" size="1.778" layer="95" rot="R180" align="top-right"/>
@@
 <instance part="CON_POUT" gate="-1" x="10.16" y="5.08"/>
 <instance part="CON_POUT" gate="-2" x="10.16" y="0"/>
+<instance part="R4" gate="G$1" x="132.08" y="24.13"/>
 </instances>
 <busses>
@@
 </segment>
 <segment>
-<pinref part="R4" gate="G$1" pin="1"/>
 <wire x1="127" y1="24.13" x2="125.73" y2="24.13" width="0.1524" layer="91"/>
 <label x="119.38" y="24.13" size="1.778" layer="95"/>
@@
 <wire x1="125.73" y1="21.59" x2="120.65" y2="21.59" width="0.1524" layer="91"/>
 <pinref part="R5" gate="G$1" pin="2"/>
+<pinref part="R4" gate="G$1" pin="1"/>
 </segment>
 <segment>
@@
 <segment>
 <wire x1="139.7" y1="10.16" x2="139.7" y2="24.13" width="0.1524" layer="91"/>
-<pinref part="R4" gate="G$1" pin="2"/>
 <wire x1="139.7" y1="24.13" x2="139.7" y2="26.67" width="0.1524" layer="91"/>
 <wire x1="139.7" y1="26.67" x2="139.7" y2="27.94" width="0.1524" layer="91"/>
-<wire x1="137.16" y1="24.13" x2="138.43" y2="24.13" width="0.1524" layer="91"/>
 <junction x="139.7" y="24.13"/>
-<wire x1="138.43" y1="24.13" x2="139.7" y2="24.13" width="0.1524" layer="91"/>
-<wire x1="138.43" y1="24.13" x2="138.43" y2="13.97" width="0.1524" layer="91"/>
-<junction x="138.43" y="24.13"/>
-<wire x1="138.43" y1="13.97" x2="120.65" y2="13.97" width="0.1524" layer="91"/>
+<wire x1="137.16" y1="24.13" x2="139.7" y2="24.13" width="0.1524" layer="91"/>
+<wire x1="137.16" y1="24.13" x2="137.16" y2="13.97" width="0.1524" layer="91"/>
+<wire x1="137.16" y1="13.97" x2="120.65" y2="13.97" width="0.1524" layer="91"/>
 <wire x1="139.7" y1="26.67" x2="144.78" y2="26.67" width="0.1524" layer="91"/>
 <junction x="139.7" y="26.67"/>
@@
 <pinref part="Q2" gate="G$1" pin="S"/>
 <pinref part="Q3" gate="G$1" pin="S"/>
-</segment>
-</net>
+<pinref part="R4" gate="G$1" pin="2"/>
+<junction x="137.16" y="24.13"/>
+</segment>
+</net>

Commit message: [ update ] sch
Other:
- note removed: "TODO: q1 sqj886ep-t1-ge3 package is powerpak-so8, not powerpak-so8-l"
Changed lines of the file:
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@@
 <text x="-5.08" y="100.33" size="1.778" layer="97">r2 = vout * r1 / 0.8 - r1</text>
 <text x="-5.08" y="97.79" size="1.778" layer="97">3.4V, 5.2V, 12V, 19.6V</text>
-<text x="119.38" y="66.04" size="1.778" layer="97">TODO: q1 sqj886ep-t1-ge3 package is powerpak-so8, not powerpak-so8-l</text>
 <text x="119.38" y="58.42" size="1.778" layer="97">NOTE: D3, D4 are B240A</text>
 <text x="163.83" y="119.38" size="1.778" layer="97">NOTE: D1, D2 are DFLS160</text>

Commit message: [ update ] sch
Other:
- note added: "https://github.com/texane/dc_converter"
- note added: "texane@gmail.com"
- moved on the sheet: C12, C13, C6, C7, C8_0, C8_1, C8_2, C8_3, C8_4, D1, D2, D3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
