File: eagle/main.sch (EAGLE design)
At the start: 43 parts, among them Q1 SQJ886EP, U1 LTC3789EGNPBF

Commit message: [ update ] sch
Other:
- note added: "master 4a76bff"
Changed lines of the file:
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@@
 <text x="133.35" y="-25.4" size="1.778" layer="97">https://github.com/texane/dc_converter</text>
 <text x="133.35" y="-29.21" size="1.778" layer="97">texane@gmail.com</text>
-<text x="133.35" y="-33.02" size="1.778" layer="97">NOTE: Q1 is SQJ886EP-T1-GE3</text>
+<text x="133.35" y="-33.02" size="1.778" layer="97">master 4a76bff</text>
 </plain>
 <instances>
