File: eagle/main.brd (EAGLE design)
At the start: 100 x 80 mm, 31 parts, among them Q1 BSS97, Q2 BSS97, Q3 BSS97, Q4 BSS97, U1 LTC3789EGNPBF

Commit message: [ update ] sch
Parts:
- removed D5, D6: 1N4148DO35-10, diode:DO35-10
- added D1, D2: (no value), diode:POWER-DI-123
- moved D3 20.3 mm to (-45.7, 52.1)
- moved D4 20.3 mm to (-25.4, 52.1)
Connections:
- net BOOST1: now also D1.C; no longer D5.C
- net BOOST2: now also D2.C; no longer D6.C
- net INTVCC: now also D1.A, D2.A; no longer D5.A, D6.A
- net N$9: now also D3.A; no longer D4.A
- net SW1: now also D3.C; no longer D4.C
- net SW2: now also D4.A; no longer D3.A
- net VOUT: now also D4.C; no longer D3.C
Changed lines of the file:
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@@
 <layer number="98" name="Guide" color="6" fill="1" visible="no" active="no"/>
 <layer number="99" name="SpiceOrder" color="7" fill="1" visible="no" active="no"/>
+<layer number="100" name="Muster" color="7" fill="1" visible="no" active="no"/>
+<layer number="101" name="Patch_Top" color="12" fill="4" visible="yes" active="yes"/>
+<layer number="102" name="Vscore" color="7" fill="1" visible="yes" active="yes"/>
+<layer number="103" name="tMap" color="7" fill="1" visible="yes" active="yes"/>
+<layer number="104" name="Name" color="16" fill="1" visible="yes" active="yes"/>
+<layer number="105" name="tPlate" color="7" fill="1" visible="yes" active="yes"/>
+<layer number="106" name="bPlate" color="7" fill="1" visible="yes" active="yes"/>
+<layer number="107" name="Crop" color="7" fill="1" visible="yes" active="yes"/>
+<layer number="116" name="Patch_BOT" color="9" fill="4" visible="yes" active="yes"/>
+<layer number="121" name="_tsilk" color="7" fill="1" visible="no" active="yes"/>
+<layer number="122" name="_bsilk" color="7" fill="1" visible="no" active="yes"/>
+<layer number="125" name="_tNames" color="7" fill="1" visible="no" active="yes"/>
+<layer number="144" name="Drill_legend" color="7" fill="1" visible="yes" active="yes"/>
+<layer number="151" name="HeatSink" color="7" fill="1" visible="yes" active="yes"/>
+<layer number="200" name="200bmp" color="1" fill="10" visible="yes" active="yes"/>
+<layer number="201" name="201bmp" color="2" fill="10" visible="yes" active="yes"/>
+<layer number="202" name="202bmp" color="3" fill="10" visible="yes" active="yes"/>
+<layer number="203" name="203bmp" color="4" fill="10" visible="yes" active="yes"/>
+<layer number="204" name="204bmp" color="5" fill="10" visible="yes" active="yes"/>
+<layer number="205" name="205bmp" color="6" fill="10" visible="yes" active="yes"/>
+<layer number="206" name="206bmp" color="7" fill="10" visible="yes" active="yes"/>
+<layer number="207" name="207bmp" color="8" fill="10" visible="yes" active="yes"/>
+<layer number="208" name="208bmp" color="9" fill="10" visible="yes" active="yes"/>
+<layer number="209" name="209bmp" color="7" fill="1" visible="yes" active="yes"/>
+<layer number="210" name="210bmp" color="7" fill="1" visible="yes" active="yes"/>
+<layer number="211" name="211bmp" color="7" fill="1" visible="yes" active="yes"/>
+<layer number="212" name="212bmp" color="7" fill="1" visible="yes" active="yes"/>
+<layer number="213" name="213bmp" color="7" fill="1" visible="yes" active="yes"/>
+<layer number="214" name="214bmp" color="7" fill="1" visible="yes" active="yes"/>
+<layer number="215" name="215bmp" color="7" fill="1" visible="yes" active="yes"/>
+<layer number="216" name="216bmp" color="7" fill="1" visible="yes" active="yes"/>
+<layer number="217" name="217bmp" color="18" fill="1" visible="no" active="no"/>
+<layer number="218" name="218bmp" color="19" fill="1" visible="no" active="no"/>
+<layer number="219" name="219bmp" color="20" fill="1" visible="no" active="no"/>
+<layer number="220" name="220bmp" color="21" fill="1" visible="no" active="no"/>
+<layer number="221" name="221bmp" color="22" fill="1" visible="no" active="no"/>
+<layer number="222" name="222bmp" color="23" fill="1" visible="no" active="no"/>
+<layer number="223" name="223bmp" color="24" fill="1" visible="no" active="no"/>
+<layer number="224" name="224bmp" color="25" fill="1" visible="no" active="no"/>
 <layer number="250" name="Descript" color="3" fill="1" visible="no" active="no"/>
 <layer number="251" name="SMDround" color="12" fill="11" visible="no" active="no"/>
+<layer number="254" name="cooling" color="7" fill="1" visible="yes" active="yes"/>
 </layers>
 <board>
@@
 <element name="C4" library="rcl" package="C1206K" value="1u" x="-35.56" y="71.12"/>
 <element name="C5" library="rcl" package="C1206K" value="4.7u" x="-40.64" y="71.12"/>
-<element name="D3" library="diode" package="DO35-10" value="1N4148DO35-10" x="-25.4" y="52.07"/>
-<element name="D4" library="diode" package="DO35-10" value="1N4148DO35-10" x="-45.72" y="52.07"/>
+<element name="D4" library="diode" package="DO35-10" value="1N4148DO35-10" x="-25.4" y="52.07"/>
+<element name="D3" library="diode" package="DO35-10" value="1N4148DO35-10" x="-45.72" y="52.07"/>
 <element name="Q1" library="transistor-fet" package="TO202" value="BSS97" x="-19.05" y="7.62"/>
 <element name="Q2" library="transistor-fet" package="TO202" value="BSS97" x="-30.48" y="7.62"/>
@@
 <element name="C8" library="rcl" package="C1206K" value="47u" x="-50.8" y="71.12"/>
 <element name="R4" library="resistor" package="R1206" value="0.01" x="-34.29" y="64.77"/>
-<element name="D5" library="diode" package="DO35-10" value="1N4148DO35-10" x="-25.4" y="58.42"/>
-<element name="D6" library="diode" package="DO35-10" value="1N4148DO35-10" x="-45.72" y="58.42"/>
 <element name="C12" library="rcl" package="C1206K" value="0.22u" x="-64.77" y="64.77"/>
 <element name="C13" library="rcl" package="C1206K" value="0.22u" x="-15.24" y="71.12"/>
@@
 <attribute name="OC_FARNELL" value="1848236" x="0" y="0" size="1.778" layer="27" display="off"/>
 </element>
+<element name="D1" library="diode" package="POWER-DI-123" value="" x="-64.77" y="-3.81"/>
+<element name="D2" library="diode" package="POWER-DI-123" value="" x="-64.77" y="-7.62"/>
 </elements>
 <signals>
@@
 <contactref element="C6" pad="1"/>
 <contactref element="Q4" pad="2"/>
-<contactref element="D3" pad="C"/>
+<contactref element="D4" pad="C"/>
 <contactref element="U1" pad="13"/>
 <contactref element="U1" pad="14"/>
@@
 <signal name="BOOST1">
 <contactref element="U1" pad="25"/>
-<contactref element="D5" pad="C"/>
 <contactref element="C12" pad="2"/>
-<wire x1="-47.0662" y1="40.3352" x2="-30.48" y2="58.42" width="0" layer="19" extent="1-1"/>
+<contactref element="D1" pad="C"/>
+<wire x1="-47.0662" y1="40.3352" x2="-66.74" y2="-3.81" width="0" layer="19" extent="1-1"/>
 <wire x1="-63.27" y1="64.77" x2="-47.0662" y2="40.3352" width="0" layer="19" extent="1-1"/>
 </signal>
 <signal name="BOOST2">
 <contactref element="U1" pad="18"/>
-<contactref element="D6" pad="C"/>
 <contactref element="C13" pad="2"/>
-<wire x1="-50.8" y1="58.42" x2="-13.74" y2="71.12" width="0" layer="19" extent="1-1"/>
-<wire x1="-47.0662" y1="35.8648" x2="-50.8" y2="58.42" width="0" layer="19" extent="1-1"/>
+<contactref element="D2" pad="C"/>
+<wire x1="-47.0662" y1="35.8648" x2="-66.74" y2="-7.62" width="0" layer="19" extent="1-1"/>
+<wire x1="-13.74" y1="71.12" x2="-47.0662" y2="35.8648" width="0" layer="19" extent="1-1"/>
 </signal>
 <signal name="TG2">
@@
 <contactref element="Q4" pad="1"/>
 <contactref element="Q3" pad="2"/>
-<contactref element="D3" pad="A"/>
+<contactref element="D4" pad="A"/>
 <contactref element="L1" pad="1"/>
 <contactref element="C13" pad="1"/>
@@
 <contactref element="Q1" pad="1"/>
 <contactref element="Q2" pad="2"/>
-<contactref element="D4" pad="C"/>
+<contactref element="D3" pad="C"/>
 <contactref element="L1" pad="2"/>
 <contactref element="C12" pad="1"/>
@@
 <contactref element="Q2" pad="1"/>
 <contactref element="R4" pad="2"/>
-<contactref element="D4" pad="A"/>
+<contactref element="D3" pad="A"/>
 <contactref element="R6" pad="2"/>
 <wire x1="-33.02" y1="2.54" x2="-44.45" y2="2.54" width="0" layer="19" extent="1-1"/>
@@
 </signal>
 <signal name="INTVCC">
-<contactref element="D5" pad="A"/>
-<contactref element="D6" pad="A"/>
 <contactref element="U1" pad="21"/>
 <contactref element="C5" pad="1"/>
-<wire x1="-40.64" y1="58.42" x2="-20.32" y2="58.42" width="0" layer="19" extent="1-1"/>
-<wire x1="-42.14" y1="71.12" x2="-40.64" y2="58.42" width="0" layer="19" extent="1-1"/>
-<wire x1="-47.0662" y1="37.7952" x2="-40.64" y2="58.42" width="0" layer="19" extent="1-1"/>
+<contactref element="D1" pad="A"/>
+<contactref element="D2" pad="A"/>
+<wire x1="-62.8" y1="-3.81" x2="-62.8" y2="-7.62" width="0" layer="19" extent="1-1"/>
+<wire x1="-47.0662" y1="37.7952" x2="-62.8" y2="-3.81" width="0" layer="19" extent="1-1"/>
+<wire x1="-42.14" y1="71.12" x2="-47.0662" y2="37.7952" width="0" layer="19" extent="1-1"/>
 </signal>
 </signals>

Commit message: [ update ] sch
Parts:
- added R12: 121K, resistor:R1206
- D3, D4: value 1N4148DO35-10 -> (none); device diode:DO35-10 -> diode:DO214AC
- Q2, Q3, Q4: value BSS97 -> (none); device transistor-fet:TO202 -> transistor-power:SO-08
- moved D4 80.2 mm to (-64.8, -17.8)
- moved D3 67.5 mm to (-64.8, -12.7)
- moved Q4 61.0 mm to (7.62, 10.2), turned to 270 degrees
- moved Q2 59.7 mm to (-82.5, -21.6)
- moved Q3 57.5 mm to (-91.4, -21.6)
Connections:
- new net N$6: R12.1, U1.28
- net BG1: now also Q2.4; no longer Q2.3
- net BG2: now also Q3.4; no longer Q3.3
- net INTVCC: now also R12.2
- net N$9: now also Q2.2, Q2.3, Q3.2, Q3.3
- net SW1: now also Q2.5, Q2.6, Q2.7, Q2.8; no longer Q2.2
- net SW2: now also Q3.5, Q3.6, Q3.7, Q3.8, Q4.2, Q4.3; no longer Q3.2
- net TG2: now also Q4.4; no longer Q4.3
- net VOUT: now also Q4.5, Q4.6, Q4.7, Q4.8; no longer Q4.2

Commit message: [ update ] sch
Parts:
- Q1: value BSS97 -> SQJ886EP; device transistor-fet:TO202 -> transistor-fet:POWERPAK-SO-08
- moved Q1 35.3 mm to (8.89, 29.2)
Connections:
- net SW1: now also Q1.2, Q1.3
- net TG1: now also Q1.4; no longer Q1.3
- net VIN: now also Q1.5-8; no longer Q1.2
Changed lines of the file:
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@@
 <setting verticaltext="up"/>
 </settings>
-<grid distance="0.05" unitdist="inch" unit="inch" style="lines" multiple="1" display="no" altdistance="0.025" altunitdist="inch" altunit="inch"/>
+<grid distance="0.05" unitdist="inch" unit="inch" style="lines" multiple="1" display="yes" altdistance="0.025" altunitdist="inch" altunit="inch"/>
 <layers>
 <layer number="1" name="Top" color="4" fill="1" visible="yes" active="yes"/>
@@
 <element name="C4" library="rcl" package="C1206K" value="1u" x="-35.56" y="71.12"/>
 <element name="C5" library="rcl" package="C1206K" value="4.7u" x="-40.64" y="71.12"/>
-<element name="Q1" library="transistor-fet" package="TO202" value="BSS97" x="-19.05" y="7.62"/>
 <element name="C6" library="rcl" package="C1206K" value="2.2u" x="-45.72" y="71.12"/>
 <element name="C7" library="rcl" package="PANASONIC_A" value="330u" x="-66.04" y="33.02"/>
@@
 <element name="Q3" library="transistor-power" package="SO-08" value="" x="-91.44" y="-21.59"/>
 <element name="Q4" library="transistor-power" package="SO-08" value="" x="7.62" y="10.16" rot="R270"/>
+<element name="Q1" library="transistor-fet" package="POWERPAK-SO-08" value="SQJ886EP" x="8.89" y="29.21"/>
 </elements>
 <signals>
@@
 <contactref element="R10" pad="1"/>
 <contactref element="C8" pad="1"/>
-<contactref element="Q1" pad="2"/>
-<wire x1="-56.032" y1="64.77" x2="-52.3" y2="71.12" width="0" layer="19" extent="1-1"/>
-<wire x1="-51.9938" y1="36.5252" x2="-56.032" y2="64.77" width="0" layer="19" extent="1-1"/>
-<wire x1="-19.05" y1="2.54" x2="-51.9938" y2="36.5252" width="0" layer="19" extent="1-1"/>
+<contactref element="Q1" pad="5-8"/>
+<wire x1="-51.9938" y1="36.5252" x2="8.89" y2="31.115" width="0" layer="19" extent="1-1"/>
+<wire x1="-56.032" y1="64.77" x2="-51.9938" y2="36.5252" width="0" layer="19" extent="1-1"/>
+<wire x1="-52.3" y1="71.12" x2="-56.032" y2="64.77" width="0" layer="19" extent="1-1"/>
 </signal>
 <signal name="SENSE-">
@@
 <signal name="TG1">
 <contactref element="U1" pad="26"/>
-<contactref element="Q1" pad="3"/>
-<wire x1="-47.0662" y1="40.9448" x2="-16.51" y2="2.54" width="0" layer="19" extent="1-1"/>
+<contactref element="Q1" pad="4"/>
+<wire x1="-47.0662" y1="40.9448" x2="10.795" y2="26.3525" width="0" layer="19" extent="1-1"/>
 </signal>
 <signal name="BG2">
@@
 <signal name="SW1">
 <contactref element="U1" pad="27"/>
-<contactref element="Q1" pad="1"/>
 <contactref element="L1" pad="2"/>
 <contactref element="C12" pad="1"/>
@@
 <contactref element="Q2" pad="6"/>
 <contactref element="Q2" pad="7"/>
+<contactref element="Q1" pad="1"/>
+<contactref element="Q1" pad="2"/>
+<contactref element="Q1" pad="3"/>
+<wire x1="8.255" y1="26.3525" x2="6.985" y2="26.3525" width="0" layer="19" extent="1-1"/>
+<wire x1="9.525" y1="26.3525" x2="8.255" y2="26.3525" width="0" layer="19" extent="1-1"/>
+<wire x1="-84.455" y1="-18.99" x2="9.525" y2="26.3525" width="0" layer="19" extent="1-1"/>
 <wire x1="-83.185" y1="-18.99" x2="-84.455" y2="-18.99" width="0" layer="19" extent="1-1"/>
 <wire x1="-81.915" y1="-18.99" x2="-83.185" y2="-18.99" width="0" layer="19" extent="1-1"/>
 <wire x1="-80.645" y1="-18.99" x2="-81.915" y2="-18.99" width="0" layer="19" extent="1-1"/>
 <wire x1="-66.82" y1="-12.7" x2="-80.645" y2="-18.99" width="0" layer="19" extent="1-1"/>
-<wire x1="-21.59" y1="2.54" x2="-66.82" y2="-12.7" width="0" layer="19" extent="1-1"/>
-<wire x1="-15.37" y1="39.37" x2="-21.59" y2="2.54" width="0" layer="19" extent="1-1"/>
-<wire x1="-47.0662" y1="41.6052" x2="-15.37" y2="39.37" width="0" layer="19" extent="1-1"/>
+<wire x1="-47.0662" y1="41.6052" x2="-66.82" y2="-12.7" width="0" layer="19" extent="1-1"/>
 <wire x1="-66.27" y1="64.77" x2="-47.0662" y2="41.6052" width="0" layer="19" extent="1-1"/>
+<wire x1="-15.37" y1="39.37" x2="-47.0662" y2="41.6052" width="0" layer="19" extent="1-1"/>
 </signal>
 <signal name="N$9">

Commit message: [ update ] sch
Parts:
- C7: value 330u -> 330UF; device rcl:PANASONIC_A -> Panasonic-EEEFT_EEEH:CAPAE1030X1050N
- moved C7 61.7 mm to (-102.9, -16.5)
Connections:
- net GND: now also C7.2; no longer C7.-
- net VOUT: now also C7.1; no longer C7.+
Other:
- board size 100 x 80 mm -> 49.2 x 49.5 mm
Changed lines of the file:
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@@
 <setting verticaltext="up"/>
 </settings>
-<grid distance="0.05" unitdist="inch" unit="inch" style="lines" multiple="1" display="yes" altdistance="0.025" altunitdist="inch" altunit="inch"/>
+<grid distance="1.27" unitdist="mm" unit="mm" style="lines" multiple="1" display="yes" altdistance="0.025" altunitdist="inch" altunit="inch"/>
 <layers>
 <layer number="1" name="Top" color="4" fill="1" visible="yes" active="yes"/>
@@
 <board>
 <plain>
-<wire x1="0" y1="0" x2="100" y2="0" width="0" layer="20"/>
-<wire x1="100" y1="0" x2="100" y2="80" width="0" layer="20"/>
-<wire x1="100" y1="80" x2="0" y2="80" width="0" layer="20"/>
-<wire x1="0" y1="80" x2="0" y2="0" width="0" layer="20"/>
+<wire x1="0" y1="0" x2="49.2" y2="0" width="0" layer="20"/>
+<wire x1="49.2" y1="0" x2="49.2" y2="49.52" width="0" layer="20"/>
+<wire x1="49.2" y1="49.52" x2="0" y2="49.52" width="0" layer="20"/>
+<wire x1="0" y1="49.52" x2="0" y2="0" width="0" layer="20"/>
 </plain>
 <attributes>
@@
 <element name="C5" library="rcl" package="C1206K" value="4.7u" x="-40.64" y="71.12"/>
 <element name="C6" library="rcl" package="C1206K" value="2.2u" x="-45.72" y="71.12"/>
-<element name="C7" library="rcl" package="PANASONIC_A" value="330u" x="-66.04" y="33.02"/>
 <element name="C8" library="rcl" package="C1206K" value="47u" x="-50.8" y="71.12"/>
 <element name="R4" library="resistor" package="R1206" value="0.01" x="-34.29" y="64.77"/>
@@
 <element name="Q4" library="transistor-power" package="SO-08" value="" x="7.62" y="10.16" rot="R270"/>
 <element name="Q1" library="transistor-fet" package="POWERPAK-SO-08" value="SQJ886EP" x="8.89" y="29.21"/>
+<element name="C7" library="Panasonic-EEEFT_EEEH" package="CAPAE1030X1050N" value="330UF" x="-102.87" y="-16.51">
+<attribute name="PACKAGE" value="CASE-G" x="-102.87" y="-16.51" size="1.778" layer="27" display="off"/>
+<attribute name="OC_NEWARK" value="31T8184" x="-102.87" y="-16.51" size="1.778" layer="27" display="off"/>
+<attribute name="TOLERANCE" value="±20 %" x="-102.87" y="-16.51" size="1.778" layer="27" display="off"/>
+<attribute name="MPN" value="EEE-FT1H331AP" x="-102.87" y="-16.51" size="1.778" layer="27" display="off"/>
+<attribute name="SUPPLIER" value="PANASONIC" x="-102.87" y="-16.51" size="1.778" layer="27" display="off"/>
+<attribute name="VOLTAGERATING" value="50V" x="-102.87" y="-16.51" size="1.778" layer="27" display="off"/>
+<attribute name="OC_FARNELL" value="1868428  " x="-102.87" y="-16.51" size="1.778" layer="27" display="off"/>
+</element>
 </elements>
 <signals>
@@
 <contactref element="R4" pad="1"/>
 <contactref element="R5" pad="2"/>
-<contactref element="C7" pad="-"/>
-<wire x1="-23.9" y1="71.12" x2="-21.82" y2="71.12" width="0" layer="19" extent="1-1"/>
-<wire x1="-28.98" y1="71.12" x2="-23.9" y2="71.12" width="0" layer="19" extent="1-1"/>
-<wire x1="-30.632" y1="64.77" x2="-28.98" y2="71.12" width="0" layer="19" extent="1-1"/>
-<wire x1="-35.712" y1="64.77" x2="-30.632" y2="64.77" width="0" layer="19" extent="1-1"/>
-<wire x1="-40.792" y1="64.77" x2="-35.712" y2="64.77" width="0" layer="19" extent="1-1"/>
-<wire x1="-43.028" y1="64.77" x2="-40.792" y2="64.77" width="0" layer="19" extent="1-1"/>
+<contactref element="C7" pad="2"/>
+<wire x1="-51.9938" y1="35.2552" x2="-98.806" y2="-16.51" width="0" layer="19" extent="1-1"/>
+<wire x1="-51.9938" y1="38.4048" x2="-51.9938" y2="35.2552" width="0" layer="19" extent="1-1"/>
+<wire x1="-51.9938" y1="39.0652" x2="-51.9938" y2="38.4048" width="0" layer="19" extent="1-1"/>
+<wire x1="-47.0662" y1="39.6748" x2="-51.9938" y2="39.0652" width="0" layer="19" extent="1-1"/>
+<wire x1="-47.0662" y1="33.9852" x2="-51.9938" y2="35.2552" width="0" layer="19" extent="1-1"/>
+<wire x1="-43.028" y1="64.77" x2="-47.0662" y2="39.6748" width="0" layer="19" extent="1-1"/>
+<wire x1="-40.792" y1="64.77" x2="-43.028" y2="64.77" width="0" layer="19" extent="1-1"/>
+<wire x1="-35.712" y1="64.77" x2="-40.792" y2="64.77" width="0" layer="19" extent="1-1"/>
+<wire x1="-30.632" y1="64.77" x2="-35.712" y2="64.77" width="0" layer="19" extent="1-1"/>
 <wire x1="-44.22" y1="71.12" x2="-43.028" y2="64.77" width="0" layer="19" extent="1-1"/>
 <wire x1="-39.14" y1="71.12" x2="-44.22" y2="71.12" width="0" layer="19" extent="1-1"/>
 <wire x1="-37.06" y1="71.12" x2="-39.14" y2="71.12" width="0" layer="19" extent="1-1"/>
 <wire x1="-49.3" y1="71.12" x2="-44.22" y2="71.12" width="0" layer="19" extent="1-1"/>
-<wire x1="-47.0662" y1="39.6748" x2="-43.028" y2="64.77" width="0" layer="19" extent="1-1"/>
-<wire x1="-51.9938" y1="39.0652" x2="-47.0662" y2="39.6748" width="0" layer="19" extent="1-1"/>
-<wire x1="-51.9938" y1="38.4048" x2="-51.9938" y2="39.0652" width="0" layer="19" extent="1-1"/>
-<wire x1="-51.9938" y1="35.2552" x2="-51.9938" y2="38.4048" width="0" layer="19" extent="1-1"/>
-<wire x1="-47.0662" y1="33.9852" x2="-51.9938" y2="35.2552" width="0" layer="19" extent="1-1"/>
-<wire x1="-67.34" y1="33.02" x2="-51.9938" y2="35.2552" width="0" layer="19" extent="1-1"/>
+<wire x1="-28.98" y1="71.12" x2="-30.632" y2="64.77" width="0" layer="19" extent="1-1"/>
+<wire x1="-23.9" y1="71.12" x2="-28.98" y2="71.12" width="0" layer="19" extent="1-1"/>
+<wire x1="-21.82" y1="71.12" x2="-23.9" y2="71.12" width="0" layer="19" extent="1-1"/>
 </signal>
 <signal name="VOUT">
@@
 <contactref element="U1" pad="11"/>
 <contactref element="U1" pad="20"/>
-<contactref element="C7" pad="+"/>
 <contactref element="C6" pad="1"/>
 <contactref element="U1" pad="13"/>
@@
 <contactref element="Q4" pad="6"/>
 <contactref element="Q4" pad="7"/>
-<wire x1="10.22" y1="10.795" x2="10.22" y2="12.065" width="0" layer="19" extent="1-1"/>
-<wire x1="10.22" y1="9.525" x2="10.22" y2="10.795" width="0" layer="19" extent="1-1"/>
-<wire x1="10.22" y1="8.255" x2="10.22" y2="9.525" width="0" layer="19" extent="1-1"/>
-<wire x1="-66.82" y1="-17.78" x2="10.22" y2="8.255" width="0" layer="19" extent="1-1"/>
-<wire x1="-64.74" y1="33.02" x2="-66.82" y2="-17.78" width="0" layer="19" extent="1-1"/>
-<wire x1="-51.9938" y1="33.9852" x2="-64.74" y2="33.02" width="0" layer="19" extent="1-1"/>
+<contactref element="C7" pad="1"/>
+<wire x1="-66.82" y1="-17.78" x2="-106.934" y2="-16.51" width="0" layer="19" extent="1-1"/>
+<wire x1="-51.9938" y1="33.9852" x2="-66.82" y2="-17.78" width="0" layer="19" extent="1-1"/>
 <wire x1="-51.9938" y1="34.5948" x2="-51.9938" y2="33.9852" width="0" layer="19" extent="1-1"/>
 <wire x1="-51.9938" y1="35.8648" x2="-51.9938" y2="34.5948" width="0" layer="19" extent="1-1"/>
@@
 <wire x1="-21.438" y1="64.77" x2="-47.22" y2="71.12" width="0" layer="19" extent="1-1"/>
 <wire x1="-15.088" y1="64.77" x2="-21.438" y2="64.77" width="0" layer="19" extent="1-1"/>
+<wire x1="10.22" y1="12.065" x2="-15.088" y2="64.77" width="0" layer="19" extent="1-1"/>
+<wire x1="10.22" y1="10.795" x2="10.22" y2="12.065" width="0" layer="19" extent="1-1"/>
+<wire x1="10.22" y1="9.525" x2="10.22" y2="10.795" width="0" layer="19" extent="1-1"/>
+<wire x1="10.22" y1="8.255" x2="10.22" y2="9.525" width="0" layer="19" extent="1-1"/>
 </signal>
 <signal name="VIN">
