File: eagle/main.brd (EAGLE design)
At the start: 49.2 x 49.5 mm, 32 parts, among them Q1 SQJ886EP, U1 LTC3789EGNPBF

Commit message: [ update ] sch
Parts:
- added C8_1, C8_2, C8_3, C8_4: 10u, rcl:C1206K
- C8_0: value 47u -> 10u
- renumbered C8 to C8_0
Connections:
- net GND: now also C8_1.2, C8_2.2, C8_3.2, C8_4.2
- net VIN: now also C8_1.1, C8_2.1, C8_3.1, C8_4.1
Changed lines of the file:
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@@
 <element name="C5" library="rcl" package="C1206K" value="4.7u" x="-40.64" y="71.12"/>
 <element name="C6" library="rcl" package="C1206K" value="2.2u" x="-45.72" y="71.12"/>
-<element name="C8" library="rcl" package="C1206K" value="47u" x="-50.8" y="71.12"/>
+<element name="C8_0" library="rcl" package="C1206K" value="10u" x="-50.8" y="71.12"/>
 <element name="R4" library="resistor" package="R1206" value="0.01" x="-34.29" y="64.77"/>
 <element name="C12" library="rcl" package="C1206K" value="0.22u" x="-64.77" y="64.77"/>
@@
 <attribute name="OC_FARNELL" value="1868428  " x="-102.87" y="-16.51" size="1.778" layer="27" display="off"/>
 </element>
+<element name="C8_1" library="rcl" package="C1206K" value="10u" x="-107.95" y="-29.21"/>
+<element name="C8_2" library="rcl" package="C1206K" value="10u" x="-107.95" y="-34.29"/>
+<element name="C8_3" library="rcl" package="C1206K" value="10u" x="-107.95" y="-39.37"/>
+<element name="C8_4" library="rcl" package="C1206K" value="10u" x="-107.95" y="-44.45"/>
 </elements>
 <signals>
@@
 <contactref element="C4" pad="1"/>
 <contactref element="C5" pad="2"/>
-<contactref element="C8" pad="2"/>
+<contactref element="C8_0" pad="2"/>
 <contactref element="C6" pad="2"/>
 <contactref element="R4" pad="1"/>
 <contactref element="R5" pad="2"/>
 <contactref element="C7" pad="2"/>
+<contactref element="C8_4" pad="2"/>
+<contactref element="C8_3" pad="2"/>
+<contactref element="C8_2" pad="2"/>
+<contactref element="C8_1" pad="2"/>
+<wire x1="-106.45" y1="-39.37" x2="-106.45" y2="-44.45" width="0" layer="19" extent="1-1"/>
+<wire x1="-106.45" y1="-34.29" x2="-106.45" y2="-39.37" width="0" layer="19" extent="1-1"/>
+<wire x1="-106.45" y1="-29.21" x2="-106.45" y2="-34.29" width="0" layer="19" extent="1-1"/>
+<wire x1="-98.806" y1="-16.51" x2="-106.45" y2="-29.21" width="0" layer="19" extent="1-1"/>
 <wire x1="-51.9938" y1="35.2552" x2="-98.806" y2="-16.51" width="0" layer="19" extent="1-1"/>
 <wire x1="-51.9938" y1="38.4048" x2="-51.9938" y2="35.2552" width="0" layer="19" extent="1-1"/>
@@
 <contactref element="U1" pad="10"/>
 <contactref element="R10" pad="1"/>
-<contactref element="C8" pad="1"/>
+<contactref element="C8_0" pad="1"/>
 <contactref element="Q1" pad="5-8"/>
-<wire x1="-51.9938" y1="36.5252" x2="8.89" y2="31.115" width="0" layer="19" extent="1-1"/>
+<contactref element="C8_4" pad="1"/>
+<contactref element="C8_3" pad="1"/>
+<contactref element="C8_2" pad="1"/>
+<contactref element="C8_1" pad="1"/>
+<wire x1="-109.45" y1="-39.37" x2="-109.45" y2="-44.45" width="0" layer="19" extent="1-1"/>
+<wire x1="-109.45" y1="-34.29" x2="-109.45" y2="-39.37" width="0" layer="19" extent="1-1"/>
+<wire x1="-109.45" y1="-29.21" x2="-109.45" y2="-34.29" width="0" layer="19" extent="1-1"/>
+<wire x1="-51.9938" y1="36.5252" x2="-109.45" y2="-29.21" width="0" layer="19" extent="1-1"/>
 <wire x1="-56.032" y1="64.77" x2="-51.9938" y2="36.5252" width="0" layer="19" extent="1-1"/>
 <wire x1="-52.3" y1="71.12" x2="-56.032" y2="64.77" width="0" layer="19" extent="1-1"/>
+<wire x1="8.89" y1="31.115" x2="-51.9938" y2="36.5252" width="0" layer="19" extent="1-1"/>
 </signal>
 <signal name="SENSE-">

Commit message: [ update ] sch
Parts:
- added CON_POW_IN, CON_POW_OUT: (no value), pinhead:1X02
- added CON_RUN: (no value), con-lstb:MA03-1
- added CON_VSEL: (no value), con-lstb:MA04-2
- added D5: BZX84, diode:SOT23
- added R13: 280K, resistor:R1206
- added R14: 65K, resistor:R1206
Connections:
- new net N$10: CON_VSEL.3, R2_3.1
- new net N$11: CON_RUN.2, R13.1
- new net N$7: CON_VSEL.5, R2_2.1
- new net N$8: CON_VSEL.7, R2_1.1
- net GND: now also CON_POW_IN.2, CON_POW_OUT.2, CON_RUN.1, D5.1, R14.1
- net RUN: now also D5.3, R13.2, R14.2
- net VFB: now also CON_VSEL.1, CON_VSEL.2, CON_VSEL.4, CON_VSEL.6, CON_VSEL.8; no longer R2_1.1, R2_2.1, R2_3.1
- net VIN: now also CON_POW_IN.1, CON_RUN.3
- net VOUT: now also CON_POW_OUT.1
Changed lines of the file:
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@@
 <element name="C8_3" library="rcl" package="C1206K" value="10u" x="-107.95" y="-39.37"/>
 <element name="C8_4" library="rcl" package="C1206K" value="10u" x="-107.95" y="-44.45"/>
+<element name="CON_VSEL" library="con-lstb" package="MA04-2" value="" x="-104.14" y="-52.07">
+<attribute name="OC_NEWARK" value="unknown" x="-104.14" y="-52.07" size="1.778" layer="27" display="off"/>
+<attribute name="MPN" value="" x="-104.14" y="-52.07" size="1.778" layer="27" display="off"/>
+<attribute name="MF" value="" x="-104.14" y="-52.07" size="1.778" layer="27" display="off"/>
+<attribute name="OC_FARNELL" value="unknown" x="-104.14" y="-52.07" size="1.778" layer="27" display="off"/>
+</element>
+<element name="CON_RUN" library="con-lstb" package="MA03-1" value="" x="-104.14" y="-60.96">
+<attribute name="OC_NEWARK" value="unknown" x="-104.14" y="-60.96" size="1.778" layer="27" display="off"/>
+<attribute name="MPN" value="" x="-104.14" y="-60.96" size="1.778" layer="27" display="off"/>
+<attribute name="MF" value="" x="-104.14" y="-60.96" size="1.778" layer="27" display="off"/>
+<attribute name="OC_FARNELL" value="unknown" x="-104.14" y="-60.96" size="1.778" layer="27" display="off"/>
+</element>
+<element name="R13" library="resistor" package="R1206" value="280K" x="-107.95" y="-72.39"/>
+<element name="R14" library="resistor" package="R1206" value="65K" x="-107.95" y="-78.74"/>
+<element name="D5" library="diode" package="SOT23" value="BZX84" x="-107.95" y="-85.09"/>
+<element name="CON_POW_IN" library="pinhead" package="1X02" value="" x="-106.68" y="-92.71"/>
+<element name="CON_POW_OUT" library="pinhead" package="1X02" value="" x="-106.68" y="-99.06"/>
 </elements>
 <signals>
@@
 <contactref element="C8_2" pad="2"/>
 <contactref element="C8_1" pad="2"/>
+<contactref element="CON_RUN" pad="1"/>
+<contactref element="D5" pad="1"/>
+<contactref element="R14" pad="1"/>
+<contactref element="CON_POW_IN" pad="2"/>
+<contactref element="CON_POW_OUT" pad="2"/>
+<wire x1="-105.41" y1="-92.71" x2="-105.41" y2="-99.06" width="0" layer="19" extent="1-1"/>
+<wire x1="-108.9" y1="-86.19" x2="-105.41" y2="-92.71" width="0" layer="19" extent="1-1"/>
+<wire x1="-109.372" y1="-78.74" x2="-108.9" y2="-86.19" width="0" layer="19" extent="1-1"/>
+<wire x1="-106.68" y1="-60.96" x2="-109.372" y2="-78.74" width="0" layer="19" extent="1-1"/>
+<wire x1="-106.45" y1="-44.45" x2="-106.68" y2="-60.96" width="0" layer="19" extent="1-1"/>
 <wire x1="-106.45" y1="-39.37" x2="-106.45" y2="-44.45" width="0" layer="19" extent="1-1"/>
 <wire x1="-106.45" y1="-34.29" x2="-106.45" y2="-39.37" width="0" layer="19" extent="1-1"/>
@@
 <contactref element="Q4" pad="7"/>
 <contactref element="C7" pad="1"/>
+<contactref element="CON_POW_OUT" pad="1"/>
+<wire x1="-106.934" y1="-16.51" x2="-107.95" y2="-99.06" width="0" layer="19" extent="1-1"/>
 <wire x1="-66.82" y1="-17.78" x2="-106.934" y2="-16.51" width="0" layer="19" extent="1-1"/>
 <wire x1="-51.9938" y1="33.9852" x2="-66.82" y2="-17.78" width="0" layer="19" extent="1-1"/>
@@
 <contactref element="C8_2" pad="1"/>
 <contactref element="C8_1" pad="1"/>
+<contactref element="CON_RUN" pad="3"/>
+<contactref element="CON_POW_IN" pad="1"/>
+<wire x1="-101.6" y1="-60.96" x2="-107.95" y2="-92.71" width="0" layer="19" extent="1-1"/>
+<wire x1="-109.45" y1="-44.45" x2="-101.6" y2="-60.96" width="0" layer="19" extent="1-1"/>
 <wire x1="-109.45" y1="-39.37" x2="-109.45" y2="-44.45" width="0" layer="19" extent="1-1"/>
 <wire x1="-109.45" y1="-34.29" x2="-109.45" y2="-39.37" width="0" layer="19" extent="1-1"/>
@@
 </signal>
 <signal name="VFB">
-<contactref element="R2_1" pad="1"/>
+<contactref element="R2_4" pad="1"/>
+<contactref element="U1" pad="1"/>
+<contactref element="CON_VSEL" pad="8"/>
+<contactref element="CON_VSEL" pad="6"/>
+<contactref element="CON_VSEL" pad="4"/>
+<contactref element="CON_VSEL" pad="2"/>
 <contactref element="R1" pad="2"/>
-<contactref element="R2_4" pad="1"/>
-<contactref element="R2_3" pad="1"/>
-<contactref element="R2_2" pad="1"/>
-<contactref element="U1" pad="1"/>
-<wire x1="-24.282" y1="64.77" x2="-17.932" y2="64.77" width="0" layer="19" extent="1-1"/>
-<wire x1="-37.948" y1="64.77" x2="-24.282" y2="64.77" width="0" layer="19" extent="1-1"/>
-<wire x1="-58.572" y1="58.42" x2="-37.948" y2="64.77" width="0" layer="19" extent="1-1"/>
-<wire x1="-64.922" y1="58.42" x2="-58.572" y2="58.42" width="0" layer="19" extent="1-1"/>
-<wire x1="-51.9938" y1="42.2148" x2="-58.572" y2="58.42" width="0" layer="19" extent="1-1"/>
+<contactref element="CON_VSEL" pad="1"/>
+<wire x1="-107.95" y1="-50.8" x2="-107.95" y2="-53.34" width="0" layer="19" extent="1-1"/>
+<wire x1="-105.41" y1="-50.8" x2="-107.95" y2="-50.8" width="0" layer="19" extent="1-1"/>
+<wire x1="-102.87" y1="-50.8" x2="-105.41" y2="-50.8" width="0" layer="19" extent="1-1"/>
+<wire x1="-100.33" y1="-50.8" x2="-102.87" y2="-50.8" width="0" layer="19" extent="1-1"/>
+<wire x1="-51.9938" y1="42.2148" x2="-100.33" y2="-50.8" width="0" layer="19" extent="1-1"/>
+<wire x1="-37.948" y1="64.77" x2="-51.9938" y2="42.2148" width="0" layer="19" extent="1-1"/>
+<wire x1="-24.282" y1="64.77" x2="-37.948" y2="64.77" width="0" layer="19" extent="1-1"/>
 </signal>
 <signal name="N$2">
@@
 <signal name="RUN">
 <contactref element="U1" pad="9"/>
+<contactref element="R13" pad="2"/>
+<contactref element="R14" pad="2"/>
+<contactref element="D5" pad="3"/>
+<wire x1="-106.528" y1="-78.74" x2="-107.95" y2="-83.99" width="0" layer="19" extent="1-1"/>
+<wire x1="-106.528" y1="-72.39" x2="-106.528" y2="-78.74" width="0" layer="19" extent="1-1"/>
+<wire x1="-51.9938" y1="37.1348" x2="-106.528" y2="-72.39" width="0" layer="19" extent="1-1"/>
 </signal>
 <signal name="INTVCC">
@@
 <wire x1="-47.0662" y1="42.2148" x2="-66.192" y2="-22.86" width="0" layer="19" extent="1-1"/>
 </signal>
+<signal name="N$8">
+<contactref element="R2_1" pad="1"/>
+<contactref element="CON_VSEL" pad="7"/>
+<wire x1="-58.572" y1="58.42" x2="-100.33" y2="-53.34" width="0" layer="19" extent="1-1"/>
+</signal>
+<signal name="N$7">
+<contactref element="R2_2" pad="1"/>
+<contactref element="CON_VSEL" pad="5"/>
+<wire x1="-64.922" y1="58.42" x2="-102.87" y2="-53.34" width="0" layer="19" extent="1-1"/>
+</signal>
+<signal name="N$10">
+<contactref element="R2_3" pad="1"/>
+<contactref element="CON_VSEL" pad="3"/>
+<wire x1="-17.932" y1="64.77" x2="-105.41" y2="-53.34" width="0" layer="19" extent="1-1"/>
+</signal>
+<signal name="N$11">
+<contactref element="CON_RUN" pad="2"/>
+<contactref element="R13" pad="1"/>
+<wire x1="-104.14" y1="-60.96" x2="-109.372" y2="-72.39" width="0" layer="19" extent="1-1"/>
+</signal>
 </signals>

Commit message: [ update ] sch
Parts:
- removed CON_POW_IN, CON_POW_OUT: (no value), pinhead:1X02
- added POW_IN, POW_OUT: (no value), con-ptr500:AK300/2
Connections:
- net GND: now also POW_IN.2, POW_OUT.2; no longer CON_POW_IN.2, CON_POW_OUT.2
- net VIN: now also POW_IN.1; no longer CON_POW_IN.1
- net VOUT: now also POW_OUT.1; no longer CON_POW_OUT.1
Changed lines of the file:
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@@
 <element name="R14" library="resistor" package="R1206" value="65K" x="-107.95" y="-78.74"/>
 <element name="D5" library="diode" package="SOT23" value="BZX84" x="-107.95" y="-85.09"/>
-<element name="CON_POW_IN" library="pinhead" package="1X02" value="" x="-106.68" y="-92.71"/>
-<element name="CON_POW_OUT" library="pinhead" package="1X02" value="" x="-106.68" y="-99.06"/>
+<element name="POW_IN" library="con-ptr500" package="AK300/2" value="" x="-116.84" y="-91.44">
+<attribute name="OC_NEWARK" value="unknown" x="-116.84" y="-91.44" size="1.778" layer="27" display="off"/>
+<attribute name="MPN" value="" x="-116.84" y="-91.44" size="1.778" layer="27" display="off"/>
+<attribute name="MF" value="" x="-116.84" y="-91.44" size="1.778" layer="27" display="off"/>
+<attribute name="OC_FARNELL" value="unknown" x="-116.84" y="-91.44" size="1.778" layer="27" display="off"/>
+</element>
+<element name="POW_OUT" library="con-ptr500" package="AK300/2" value="" x="-128.27" y="-91.44">
+<attribute name="OC_NEWARK" value="unknown" x="-128.27" y="-91.44" size="1.778" layer="27" display="off"/>
+<attribute name="MPN" value="" x="-128.27" y="-91.44" size="1.778" layer="27" display="off"/>
+<attribute name="MF" value="" x="-128.27" y="-91.44" size="1.778" layer="27" display="off"/>
+<attribute name="OC_FARNELL" value="unknown" x="-128.27" y="-91.44" size="1.778" layer="27" display="off"/>
+</element>
 </elements>
 <signals>
@@
 <contactref element="D5" pad="1"/>
 <contactref element="R14" pad="1"/>
-<contactref element="CON_POW_IN" pad="2"/>
-<contactref element="CON_POW_OUT" pad="2"/>
-<wire x1="-105.41" y1="-92.71" x2="-105.41" y2="-99.06" width="0" layer="19" extent="1-1"/>
-<wire x1="-108.9" y1="-86.19" x2="-105.41" y2="-92.71" width="0" layer="19" extent="1-1"/>
+<contactref element="POW_IN" pad="2"/>
+<contactref element="POW_OUT" pad="2"/>
+<wire x1="-114.3508" y1="-91.44" x2="-125.7808" y2="-91.44" width="0" layer="19" extent="1-1"/>
+<wire x1="-108.9" y1="-86.19" x2="-114.3508" y2="-91.44" width="0" layer="19" extent="1-1"/>
 <wire x1="-109.372" y1="-78.74" x2="-108.9" y2="-86.19" width="0" layer="19" extent="1-1"/>
 <wire x1="-106.68" y1="-60.96" x2="-109.372" y2="-78.74" width="0" layer="19" extent="1-1"/>
@@
 <contactref element="Q4" pad="7"/>
 <contactref element="C7" pad="1"/>
-<contactref element="CON_POW_OUT" pad="1"/>
-<wire x1="-106.934" y1="-16.51" x2="-107.95" y2="-99.06" width="0" layer="19" extent="1-1"/>
+<contactref element="POW_OUT" pad="1"/>
+<wire x1="-106.934" y1="-16.51" x2="-130.7846" y2="-91.44" width="0" layer="19" extent="1-1"/>
 <wire x1="-66.82" y1="-17.78" x2="-106.934" y2="-16.51" width="0" layer="19" extent="1-1"/>
 <wire x1="-51.9938" y1="33.9852" x2="-66.82" y2="-17.78" width="0" layer="19" extent="1-1"/>
@@
 <contactref element="C8_1" pad="1"/>
 <contactref element="CON_RUN" pad="3"/>
-<contactref element="CON_POW_IN" pad="1"/>
-<wire x1="-101.6" y1="-60.96" x2="-107.95" y2="-92.71" width="0" layer="19" extent="1-1"/>
+<contactref element="POW_IN" pad="1"/>
+<wire x1="-101.6" y1="-60.96" x2="-119.3546" y2="-91.44" width="0" layer="19" extent="1-1"/>
 <wire x1="-109.45" y1="-44.45" x2="-101.6" y2="-60.96" width="0" layer="19" extent="1-1"/>
 <wire x1="-109.45" y1="-39.37" x2="-109.45" y2="-44.45" width="0" layer="19" extent="1-1"/>

Commit message: [ update ] sch
Parts:
- removed POW_IN, POW_OUT: (no value), con-ptr500:AK300/2
- added CON_PIN, CON_POUT: (no value), con-ptr500:AK300/2
- moved CON_VSEL 154.0 mm to (39.4, 3.81), turned to 180 degrees
- moved C7 150.5 mm to (43.2, 19.7), turned to 270 degrees
- moved D5 146.7 mm to (8.26, 4.45)
- moved R14 145.9 mm to (8.26, 9.53), turned to 270 degrees
- moved R13 140.1 mm to (5.71, 9.53), turned to 270 degrees
- moved Q3 131.0 mm to (29.8, 27.9)
- moved C8_4 129.6 mm to (1.27, 25.4), turned to 270 degrees
- moved C8_3 129.2 mm to (3.81, 25.4), turned to 270 degrees
- moved C8_1 129.0 mm to (8.89, 25.4), turned to 270 degrees
- moved C8_2 128.9 mm to (6.35, 25.4), turned to 270 degrees
- moved CON_RUN 127.5 mm to (2.54, 8.89), turned to 270 degrees
- moved Q2 115.3 mm to (21.6, 27.9)
- moved R2_2 114.2 mm to (40.0, 10.2), turned to 90 degrees
- moved D4 114.2 mm to (38.1, 31.8), turned to 180 degrees
- moved C12 109.4 mm to (24.8, 1.91), turned to 180 degrees
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Connections:
- net GND: now also CON_PIN.2, CON_POUT.2; no longer POW_IN.2, POW_OUT.2
- net VIN: now also CON_PIN.1; no longer POW_IN.1
- net VOUT: now also CON_POUT.1; no longer POW_OUT.1
Routing:
- added copper zone on layer 1, net GND
- added copper zone on layer 16, net GND
- added copper zone on layer 1, net N$9
- added copper zone on layer 1, net SW1
- added copper zone on layer 1, net SW2
- added copper zone on layer 1, net VIN
- added copper zone on layer 1, net VOUT
