File: eagle/main.brd (EAGLE design)
At the start: 49.5 x 49.5 mm, 43 parts, among them Q1 SQJ886EP, U1 LTC3789EGNPBF

Commit message: [ update ] sch
Parts:
- Q1: device transistor-fet:POWERPAK-SO-08 -> transistor-fet:POWERPAK-SO-08L
Changed lines of the file:
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@@
 <element name="Q3" library="transistor-power" package="SO-08" value="" x="29.845" y="28.575"/>
 <element name="Q4" library="transistor-power" package="SO-08" value="" x="38.1" y="36.83" rot="R270"/>
-<element name="Q1" library="transistor-fet" package="POWERPAK-SO-08" value="SQJ886EP" x="11.43" y="36.83" rot="R90"/>
+<element name="Q1" library="transistor-fet" package="POWERPAK-SO-08L" value="SQJ886EP" x="11.43" y="36.83" rot="R90"/>
 <element name="C7" library="Panasonic-EEEFT_EEEH" package="CAPAE1030X1050N" value="330UF" x="43.18" y="22.5425" rot="R270">
 <attribute name="PACKAGE" value="CASE-G" x="43.18" y="22.5425" size="1.778" layer="27" rot="R270" display="off"/>
@@
 <contactref element="U1" pad="26"/>
 <contactref element="Q1" pad="4"/>
-<wire x1="14.2875" y1="38.735" x2="16.1925" y2="38.735" width="0.6096" layer="1"/>
+<wire x1="14.4875" y1="38.735" x2="16.1925" y2="38.735" width="0.6096" layer="1"/>
 <via x="16.1925" y="38.735" extent="1-16" drill="0.5"/>
 <wire x1="16.1925" y1="38.735" x2="16.1925" y2="11.1125" width="0.4064" layer="16"/>

Commit message: [ update ] sch
Other:
- board text added: "+"
- board text added: "-"
- board text added: "buck boost converter"
- board text added: "revision"

Commit message: [ update ] sch
Other:
- board text added: "master 4a76bff"
- board text removed: "revision"
Changed lines of the file:
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@@
 <text x="48.895" y="40.005" size="0.6096" layer="25" font="vector" ratio="18" align="center">-</text>
 <text x="0.9525" y="32.0675" size="0.6096" layer="25" font="vector" ratio="18" align="center-left">buck boost converter</text>
-<text x="0.9525" y="31.115" size="0.6096" layer="25" font="vector" ratio="18" align="center-left">revision</text>
+<text x="0.9525" y="31.115" size="0.6096" layer="25" font="vector" ratio="18" align="center-left">master 4a76bff</text>
 </plain>
 <attributes>
